File: Pulse-Monitor.sch (KiCad schematic (older format))
At the start: 4 parts

Commit message: Documentation updates
Parts:
- removed IC?: MAX30100, OptoDevice:Maxim_OLGA-14_3.3x5.6mm_P0.8mm, symbol Sensor:MAX30100
- added IC?: PulseSensor, OptoDevice:Maxim_OLGA-14_3.3x5.6mm_P0.8mm, symbol Sensor:PulseSensor
Connections:
- net labels removed: Interrupt
- wire segments 27 -> 22
Changed lines of the file:
@@
 	0    -1   -1   0
 $EndComp
-$Comp
-L Sensor:MAX30100 IC?
-U 1 1 655686DB
-P 7350 4150
-F 0 "IC?" H 7880 4196 50  0001 L CNN
-F 1 "MAX30100" H 7250 4150 50  0000 L CNN
-F 2 "OptoDevice:Maxim_OLGA-14_3.3x5.6mm_P0.8mm" H 7200 5050 50  0001 C CNN
-F 3 "https://datasheets.maximintegrated.com/en/ds/MAX30102.pdf" H 7000 4400 50  0001 C CNN
-	1    7350 4150
-	1    0    0    -1
-$EndComp
-$Comp
-L MCU_Module:Arduino_Nano A?
-U 1 1 65570915
-P 4800 4000
-F 0 "A?" H 5980 3896 50  0001 L CNN
-F 1 "Arduino_Nano" H 4850 3850 50  0000 L CNN
-F 2 "Module:Arduino_Nano" V 5050 3850 50  0001 C CIN
-F 3 "https://www.arduino.cc/en/uploads/Main/ArduinoNanoManual23.pdf" V 5050 3850 50  0001 C CNN
-	1    4800 4000
-	1    0    0    -1
-$EndComp
-Wire Wire Line
-	5150 3650 5150 3550
-Wire Wire Line
-	5150 3550 6050 3550
-Wire Wire Line
-	6050 3550 6050 4350
-Wire Wire Line
-	6050 4350 6750 4350
-Wire Wire Line
-	6750 4200 6200 4200
-Wire Wire Line
-	6200 3400 5050 3400
-Wire Wire Line
-	5050 3400 5050 3650
-Wire Wire Line
-	6200 3400 6200 4200
-Wire Wire Line
-	5750 3650 5750 3600
-Wire Wire Line
-	5750 3600 6650 3600
-Wire Wire Line
-	6650 3600 6650 3900
-Wire Wire Line
-	6650 3900 6750 3900
-Wire Wire Line
-	4750 4800 6300 4800
-Wire Wire Line
-	6300 4800 6300 4050
-Wire Wire Line
-	6300 4050 6750 4050
-Text GLabel 6700 4500 0    50   Input ~ 0
-Interrupt
-Wire Wire Line
-	6750 4500 6700 4500
 Wire Wire Line
 	4350 3400 4350 3550
@@
 	4450 3550 4450 3650
 Wire Wire Line
-	4650 3400 4650 3550
+	4650 3400 4650 3500
 Wire Wire Line
 	4650 3550 4550 3550
@@
 Wire Wire Line
 	6750 5000 4750 5000
-Wire Wire Line
-	4750 4650 4750 4800
-Connection ~ 4750 4800
-Wire Wire Line
-	4750 4800 4750 5000
 $Comp
 L Device:Speaker LS?
@@
 Wire Wire Line
 	6750 4900 5450 4900
+$Comp
+L Sensor:PulseSensor IC?
+U 1 1 6567EC4C
+P 7050 4300
+F 0 "IC?" H 7469 4346 50  0001 L CNN
+F 1 "PulseSensor" H 7469 4300 50  0000 L CNN
+F 2 "OptoDevice:Maxim_OLGA-14_3.3x5.6mm_P0.8mm" H 6900 5200 50  0001 C CNN
+F 3 "https://datasheets.maximintegrated.com/en/ds/MAX30102.pdf" H 6700 4550 50  0001 C CNN
+	1    7050 4300
+	1    0    0    -1
+$EndComp
 Wire Wire Line
 	5450 4900 5450 4650
+Wire Wire Line
+	4750 3650 4750 3600
+Wire Wire Line
+	4750 3600 6550 3600
+$Comp
+L MCU_Module:Arduino_Nano A?
+U 1 1 65570915
+P 4800 4000
+F 0 "A?" H 5980 3896 50  0001 L CNN
+F 1 "Arduino_Nano" H 4850 3850 50  0000 L CNN
+F 2 "Module:Arduino_Nano" V 5050 3850 50  0001 C CIN
+F 3 "https://www.arduino.cc/en/uploads/Main/ArduinoNanoManual23.pdf" V 5050 3850 50  0001 C CNN
+	1    4800 4000
+	1    0    0    -1
+$EndComp
+Wire Wire Line
+	6550 4300 6700 4300
+Wire Wire Line
+	6550 3600 6550 4300
+Wire Wire Line
+	6700 4400 6600 4400
+Wire Wire Line
+	6600 4400 6600 3500
+Wire Wire Line
+	6600 3500 4650 3500
+Connection ~ 4650 3500
+Wire Wire Line
+	4650 3500 4650 3550
+Wire Wire Line
+	6700 4200 6650 4200
+Wire Wire Line
+	6650 4200 6650 3550
+Wire Wire Line
+	6650 3550 5550 3550
+Wire Wire Line
+	5550 3550 5550 3650
+Wire Wire Line
+	4750 4650 4750 5000
 $EndSCHEMATC
